File: KiboOne.sch (KiCad schematic (older format))
At the start: 137 parts, among them J1 USB_C_Receptacle, SW1 \\, SW10 4, SW11 3, SW12 2, SW13 1, SW14 esc, SW15 del, SW16 ], SW17 [, SW18 P, SW19 O, SW2 =, SW20 I, SW21 U, SW22 Y, SW23 T, SW24 R, SW25 E, SW26 W, SW27 Q, SW28 ⇥, SW29 return, SW3 -, SW30 ', SW31 ;, SW32 L, SW33 K, SW34 J, SW35 H, SW36 G, SW37 F, SW38 D, SW39 S, SW4 0, SW40 A, SW41 cmd1, SW42 /, SW43 ↑, SW44 ., SW45 ,, SW46 M, SW47 N, SW48 B, SW49 V, SW5 9, SW50 C, SW51 X, SW52 Z, SW53 tilde, SW54 shift, SW55 →, SW56 ↓, SW57 ←, SW58 cmd3, SW59 space, SW6 8, SW60 Fn, SW61 cmd2, SW62 ⌥, SW63 ctrl, SW7 7, SW8 6, SW9 5, U1 ATmega32U4-AU, Y1 16 MHz

Commit message: Basic routing, some logo work
Parts:
- D1: renamed from D61; footprint Diode_SMD:D_MiniMELF_Handsoldering -> Diode_SMD:D_MiniMELF
- D10: renamed from D12; footprint Diode_SMD:D_MiniMELF_Handsoldering -> Diode_SMD:D_MiniMELF
- D11: renamed from D20; footprint Diode_SMD:D_MiniMELF_Handsoldering -> Diode_SMD:D_MiniMELF
- D12: renamed from D28; footprint Diode_SMD:D_MiniMELF_Handsoldering -> Diode_SMD:D_MiniMELF
- D13: renamed from D36; footprint Diode_SMD:D_MiniMELF_Handsoldering -> Diode_SMD:D_MiniMELF
- D14: renamed from D44; footprint Diode_SMD:D_MiniMELF_Handsoldering -> Diode_SMD:D_MiniMELF
- D15: renamed from D62; footprint Diode_SMD:D_MiniMELF_Handsoldering -> Diode_SMD:D_MiniMELF
- D16: renamed from D54; footprint Diode_SMD:D_MiniMELF_Handsoldering -> Diode_SMD:D_MiniMELF
- D17: renamed from D46; footprint Diode_SMD:D_MiniMELF_Handsoldering -> Diode_SMD:D_MiniMELF
- D18: renamed from D38; footprint Diode_SMD:D_MiniMELF_Handsoldering -> Diode_SMD:D_MiniMELF
- D19: renamed from D30; footprint Diode_SMD:D_MiniMELF_Handsoldering -> Diode_SMD:D_MiniMELF
- D2: renamed from D53; footprint Diode_SMD:D_MiniMELF_Handsoldering -> Diode_SMD:D_MiniMELF
- D20: renamed from D22; footprint Diode_SMD:D_MiniMELF_Handsoldering -> Diode_SMD:D_MiniMELF
- D21: renamed from D14; footprint Diode_SMD:D_MiniMELF_Handsoldering -> Diode_SMD:D_MiniMELF
- D22: renamed from D6; footprint Diode_SMD:D_MiniMELF_Handsoldering -> Diode_SMD:D_MiniMELF
- D23: renamed from D3; footprint Diode_SMD:D_MiniMELF_Handsoldering -> Diode_SMD:D_MiniMELF
- D24: renamed from D11; footprint Diode_SMD:D_MiniMELF_Handsoldering -> Diode_SMD:D_MiniMELF
- D25: renamed from D19; footprint Diode_SMD:D_MiniMELF_Handsoldering -> Diode_SMD:D_MiniMELF
- D26: renamed from D27; footprint Diode_SMD:D_MiniMELF_Handsoldering -> Diode_SMD:D_MiniMELF
- D27: renamed from D35; footprint Diode_SMD:D_MiniMELF_Handsoldering -> Diode_SMD:D_MiniMELF
- D28: renamed from D43; footprint Diode_SMD:D_MiniMELF_Handsoldering -> Diode_SMD:D_MiniMELF
- D29: renamed from D55; footprint Diode_SMD:D_MiniMELF_Handsoldering -> Diode_SMD:D_MiniMELF
- D3: renamed from D45; footprint Diode_SMD:D_MiniMELF_Handsoldering -> Diode_SMD:D_MiniMELF
- D30: renamed from D47; footprint Diode_SMD:D_MiniMELF_Handsoldering -> Diode_SMD:D_MiniMELF
- D31: renamed from D39; footprint Diode_SMD:D_MiniMELF_Handsoldering -> Diode_SMD:D_MiniMELF
- D32: renamed from D31; footprint Diode_SMD:D_MiniMELF_Handsoldering -> Diode_SMD:D_MiniMELF
- D33: renamed from D23; footprint Diode_SMD:D_MiniMELF_Handsoldering -> Diode_SMD:D_MiniMELF
- D34: renamed from D15; footprint Diode_SMD:D_MiniMELF_Handsoldering -> Diode_SMD:D_MiniMELF
- D35: renamed from D7; footprint Diode_SMD:D_MiniMELF_Handsoldering -> Diode_SMD:D_MiniMELF
- D36: renamed from D2; footprint Diode_SMD:D_MiniMELF_Handsoldering -> Diode_SMD:D_MiniMELF
- D37: renamed from D10; footprint Diode_SMD:D_MiniMELF_Handsoldering -> Diode_SMD:D_MiniMELF
- D38: renamed from D18; footprint Diode_SMD:D_MiniMELF_Handsoldering -> Diode_SMD:D_MiniMELF
- D39: renamed from D26; footprint Diode_SMD:D_MiniMELF_Handsoldering -> Diode_SMD:D_MiniMELF
- D4: renamed from D37; footprint Diode_SMD:D_MiniMELF_Handsoldering -> Diode_SMD:D_MiniMELF
- D40: renamed from D34; footprint Diode_SMD:D_MiniMELF_Handsoldering -> Diode_SMD:D_MiniMELF
- D41: renamed from D42; footprint Diode_SMD:D_MiniMELF_Handsoldering -> Diode_SMD:D_MiniMELF
- D42: renamed from D63; footprint Diode_SMD:D_MiniMELF_Handsoldering -> Diode_SMD:D_MiniMELF
- D43: renamed from D57; footprint Diode_SMD:D_MiniMELF_Handsoldering -> Diode_SMD:D_MiniMELF
- D44: renamed from D40; footprint Diode_SMD:D_MiniMELF_Handsoldering -> Diode_SMD:D_MiniMELF
- D45: renamed from D32; footprint Diode_SMD:D_MiniMELF_Handsoldering -> Diode_SMD:D_MiniMELF
- D46: renamed from D24; footprint Diode_SMD:D_MiniMELF_Handsoldering -> Diode_SMD:D_MiniMELF
- D47: renamed from D16; footprint Diode_SMD:D_MiniMELF_Handsoldering -> Diode_SMD:D_MiniMELF
- D48: renamed from D8; footprint Diode_SMD:D_MiniMELF_Handsoldering -> Diode_SMD:D_MiniMELF
- D49: renamed from D1; footprint Diode_SMD:D_MiniMELF_Handsoldering -> Diode_SMD:D_MiniMELF
- D5: renamed from D29; footprint Diode_SMD:D_MiniMELF_Handsoldering -> Diode_SMD:D_MiniMELF
- D50: renamed from D9; footprint Diode_SMD:D_MiniMELF_Handsoldering -> Diode_SMD:D_MiniMELF
- D51: renamed from D17; footprint Diode_SMD:D_MiniMELF_Handsoldering -> Diode_SMD:D_MiniMELF
- D52: renamed from D25; footprint Diode_SMD:D_MiniMELF_Handsoldering -> Diode_SMD:D_MiniMELF
- D53: renamed from D33; footprint Diode_SMD:D_MiniMELF_Handsoldering -> Diode_SMD:D_MiniMELF
- D54: renamed from D41; footprint Diode_SMD:D_MiniMELF_Handsoldering -> Diode_SMD:D_MiniMELF
- D55: renamed from D60; footprint Diode_SMD:D_MiniMELF_Handsoldering -> Diode_SMD:D_MiniMELF
- D56: renamed from D59; footprint Diode_SMD:D_MiniMELF_Handsoldering -> Diode_SMD:D_MiniMELF
- D57: renamed from D58; footprint Diode_SMD:D_MiniMELF_Handsoldering -> Diode_SMD:D_MiniMELF
- D58: renamed from D48; footprint Diode_SMD:D_MiniMELF_Handsoldering -> Diode_SMD:D_MiniMELF
- D59: renamed from D56; footprint Diode_SMD:D_MiniMELF_Handsoldering -> Diode_SMD:D_MiniMELF
- D6: renamed from D21; footprint Diode_SMD:D_MiniMELF_Handsoldering -> Diode_SMD:D_MiniMELF
- D60: renamed from D49; footprint Diode_SMD:D_MiniMELF_Handsoldering -> Diode_SMD:D_MiniMELF
- D61: renamed from D50; footprint Diode_SMD:D_MiniMELF_Handsoldering -> Diode_SMD:D_MiniMELF
- D62: renamed from D51; footprint Diode_SMD:D_MiniMELF_Handsoldering -> Diode_SMD:D_MiniMELF
- D63: renamed from D52; footprint Diode_SMD:D_MiniMELF_Handsoldering -> Diode_SMD:D_MiniMELF
- D7: renamed from D13; footprint Diode_SMD:D_MiniMELF_Handsoldering -> Diode_SMD:D_MiniMELF
- D8: renamed from D5; footprint Diode_SMD:D_MiniMELF_Handsoldering -> Diode_SMD:D_MiniMELF
- D9: renamed from D4; footprint Diode_SMD:D_MiniMELF_Handsoldering -> Diode_SMD:D_MiniMELF
- SW61: footprint Button_Switch_Keyboard:SW_Matias_1.50u -> Button_Switch_Keyboard:SW_Matias_1.75u
- SW63: footprint Button_Switch_Keyboard:SW_Matias_1.25u -> Button_Switch_Keyboard:SW_Matias_1.50u
Connections:
- net labels added: D1+, D1-

Commit message: Various faffing about
Connections:
- wire segments 386 -> 449
