File: KiboOne.kicad_pcb (KiCad board)
At the start: 2 copper layers, 304.8 x 100 mm, 137 parts, among them J1 USB_C_Receptacle, SW1 \, SW10 4, SW11 3, SW12 2, SW13 1, SW14 esc, SW15 del, SW16 ], SW17 [, SW18 P, SW19 O, SW2 =, SW20 I, SW21 U, SW22 Y, SW23 T, SW24 R, SW25 E, SW26 W, SW27 Q, SW28 ⇥, SW29 return, SW3 -, SW30 ', SW31 ;, SW32 L, SW33 K, SW34 J, SW35 H, SW36 G, SW37 F, SW38 D, SW39 S, SW4 0, SW40 A, SW41 cmd1, SW42 /, SW43 ↑, SW44 ., SW45 ,, SW46 M, SW47 N, SW48 B, SW49 V, SW5 9, SW50 C, SW51 X, SW52 Z, SW53 tilde, SW54 shift, SW55 →, SW56 ↓, SW57 ←, SW58 cmd3, SW59 space, SW6 8, SW60 Fn, SW61 cmd2, SW62 ⌥, SW63 ctrl, SW7 7, SW8 6, SW9 5, U1 ATmega32U4-AU, Y1 16 MHz

Commit message: Basic routing, some logo work
Parts:
- D1, D10, D11, D12, D13, D14, D15, D16, D17, D18, D19, D2, D20, D21, D22, D23, D24, D25, D26, D27, D28, D29, D3, D30, D31, D32, D33, D34, D35, D36, D37, D38, D39, D4, D40, D41, D42, D43, D44, D45, D46, D47, D48, D49, D5, D50, D51, D52, D53, D54, D55, D56, D57, D58, D59, D6, D60, D61, D62, D63, D7, D8, D9: footprint Diode_SMD:D_MiniMELF_Handsoldering -> Diode_SMD:D_MiniMELF; moved to B.Cu
- SW61: footprint Button_Switch_Keyboard:SW_Matias_1.50u -> Button_Switch_Keyboard:SW_Matias_1.75u
- SW63: footprint Button_Switch_Keyboard:SW_Matias_1.25u -> Button_Switch_Keyboard:SW_Matias_1.50u
- moved D42 272.5 mm to (350.0, 160.2), turned to 270 degrees
- moved D63 263.0 mm to (83.3, 179.2), turned to 270 degrees
- moved D54 250.3 mm to (78.6, 160.2), turned to 270 degrees
- moved D62 247.0 mm to (109.5, 179.2), turned to 270 degrees
- moved D43 246.8 mm to (326.2, 164.9), turned to 270 degrees
- moved D53 235.4 mm to (102.4, 160.2), turned to 270 degrees
- moved D44 226.9 mm to (302.4, 160.2), turned to 270 degrees
- moved D61 225.8 mm to (138.1, 179.2), turned to 270 degrees
- moved D40 191.0 mm to (107.2, 141.1), turned to 270 degrees
- moved D1 189.6 mm to (354.8, 103.0), turned to 270 degrees
- moved D17 180.2 mm to (311.9, 122.1), turned to 270 degrees
- moved D39 167.1 mm to (126.2, 141.1), turned to 270 degrees
- moved D33 163.0 mm to (259.6, 141.1), turned to 270 degrees
- moved D2 161.9 mm to (335.8, 103.0), turned to 270 degrees
- moved D18 153.1 mm to (292.9, 122.1), turned to 270 degrees
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Connections:
- net Net-(J1-PadA6) renamed /D1+
- net Net-(J1-PadA7) renamed /D1-
- D1 pad 2: Row1 -> Row5
- D10 pad 2: Row2 -> Row4
- D11 pad 2: Row3 -> Row4
- D13 pad 2: Row5 -> Row4
- D14 pad 2: Row6 -> Row4
- D15 pad 2: Row7 -> Row6
- D16 pad 2: Row8 -> Row6
- D17 pad 2: Row1 -> Row6
- D18 pad 2: Row2 -> Row6
- D19 pad 2: Row3 -> Row6
- D2 pad 2: Row2 -> Row5
- D20 pad 2: Row4 -> Row6
- D21 pad 2: Row5 -> Row6
- D23 pad 2: Row7 -> Row3
- D24 pad 2: Row8 -> Row3
- D25 pad 2: Row1 -> Row3
- D26 pad 2: Row2 -> Row3
- D28 pad 2: Row4 -> Row3
- D29 pad 2: Row5 -> Row7
- D3 pad 2: Row3 -> Row5
- D30 pad 2: Row6 -> Row7
- D32 pad 2: Row8 -> Row7
- D33 pad 2: Row1 -> Row7
- D34 pad 2: Row2 -> Row7
- D35 pad 2: Row3 -> Row7
- D36 pad 2: Row4 -> Row2
- D37 pad 2: Row5 -> Row2
- D38 pad 2: Row6 -> Row2
- D39 pad 2: Row7 -> Row2
- D4 pad 2: Row4 -> Row5
- D40 pad 2: Row8 -> Row2
- D41 pad 2: Row1 -> Row2
- D42 pad 2: Row2 -> Row7
- D43 pad 2: Row3 -> Row1
- D44 pad 2: Row4 -> Row8
- D45 pad 2: Row5 -> Row8
- D46 pad 2: Row6 -> Row8
- D47 pad 2: Row7 -> Row8
- D50 pad 2: Row2 -> Row1
- D51 pad 2: Row3 -> Row1
- D52 pad 2: Row4 -> Row1
- D53 pad 2: Row5 -> Row1
- D54 pad 2: Row6 -> Row1
- D55 pad 2: Row7 -> Row4
- D56 pad 2: Row8 -> Row3
- D57 pad 2: Row1 -> Row2
- D58 pad 2: Row2 -> Row8
- D59 pad 2: Row3 -> Row8
- D6 pad 2: Row6 -> Row5
- D60 pad 2: Row4 -> Row1
- D61 pad 2: Row5 -> Row2
- D62 pad 2: Row6 -> Row3
- D63 pad 2: Row7 -> Row4
- D7 pad 2: Row7 -> Row5
- D8 pad 2: Row8 -> Row5
- D9 pad 2: Row1 -> Row4
- SW1 pad 1: Net-(D61-Pad1) -> Net-(D1-Pad1)
- SW10 pad 1: Net-(D12-Pad1) -> Net-(D10-Pad1)
- SW11 pad 1: Net-(D20-Pad1) -> Net-(D11-Pad1)
- SW12 pad 1: Net-(D28-Pad1) -> Net-(D12-Pad1)
- SW13 pad 1: Net-(D36-Pad1) -> Net-(D13-Pad1)
- SW14 pad 1: Net-(D44-Pad1) -> Net-(D14-Pad1)
- SW15 pad 1: Net-(D62-Pad1) -> Net-(D15-Pad1)
- SW16 pad 1: Net-(D54-Pad1) -> Net-(D16-Pad1)
- SW17 pad 1: Net-(D46-Pad1) -> Net-(D17-Pad1)
- SW18 pad 1: Net-(D38-Pad1) -> Net-(D18-Pad1)
- SW19 pad 1: Net-(D30-Pad1) -> Net-(D19-Pad1)
- SW2 pad 1: Net-(D53-Pad1) -> Net-(D2-Pad1)
- SW20 pad 1: Net-(D22-Pad1) -> Net-(D20-Pad1)
- SW21 pad 1: Net-(D14-Pad1) -> Net-(D21-Pad1)
- SW22 pad 1: Net-(D6-Pad1) -> Net-(D22-Pad1)
- SW23 pad 1: Net-(D3-Pad1) -> Net-(D23-Pad1)
- SW24 pad 1: Net-(D11-Pad1) -> Net-(D24-Pad1)
- SW25 pad 1: Net-(D19-Pad1) -> Net-(D25-Pad1)
- SW26 pad 1: Net-(D27-Pad1) -> Net-(D26-Pad1)
- SW27 pad 1: Net-(D35-Pad1) -> Net-(D27-Pad1)
- SW28 pad 1: Net-(D43-Pad1) -> Net-(D28-Pad1)
- SW29 pad 1: Net-(D55-Pad1) -> Net-(D29-Pad1)
- SW3 pad 1: Net-(D45-Pad1) -> Net-(D3-Pad1)
- SW30 pad 1: Net-(D47-Pad1) -> Net-(D30-Pad1)
- SW31 pad 1: Net-(D39-Pad1) -> Net-(D31-Pad1)
- SW32 pad 1: Net-(D31-Pad1) -> Net-(D32-Pad1)
- SW33 pad 1: Net-(D23-Pad1) -> Net-(D33-Pad1)
- SW34 pad 1: Net-(D15-Pad1) -> Net-(D34-Pad1)
- SW35 pad 1: Net-(D7-Pad1) -> Net-(D35-Pad1)
- SW36 pad 1: Net-(D2-Pad1) -> Net-(D36-Pad1)
- SW37 pad 1: Net-(D10-Pad1) -> Net-(D37-Pad1)
- SW38 pad 1: Net-(D18-Pad1) -> Net-(D38-Pad1)
- SW39 pad 1: Net-(D26-Pad1) -> Net-(D39-Pad1)
- SW4 pad 1: Net-(D37-Pad1) -> Net-(D4-Pad1)
- SW40 pad 1: Net-(D34-Pad1) -> Net-(D40-Pad1)
- SW41 pad 1: Net-(D42-Pad1) -> Net-(D41-Pad1)
- SW42 pad 1: Net-(D63-Pad1) -> Net-(D42-Pad1)
- SW43 pad 1: Net-(D57-Pad1) -> Net-(D43-Pad1)
- SW44 pad 1: Net-(D40-Pad1) -> Net-(D44-Pad1)
- SW45 pad 1: Net-(D32-Pad1) -> Net-(D45-Pad1)
- SW46 pad 1: Net-(D24-Pad1) -> Net-(D46-Pad1)
- SW47 pad 1: Net-(D16-Pad1) -> Net-(D47-Pad1)
- SW48 pad 1: Net-(D8-Pad1) -> Net-(D48-Pad1)
- SW49 pad 1: Net-(D1-Pad1) -> Net-(D49-Pad1)
- SW5 pad 1: Net-(D29-Pad1) -> Net-(D5-Pad1)
- SW50 pad 1: Net-(D9-Pad1) -> Net-(D50-Pad1)
- SW51 pad 1: Net-(D17-Pad1) -> Net-(D51-Pad1)
- SW52 pad 1: Net-(D25-Pad1) -> Net-(D52-Pad1)
- SW53 pad 1: Net-(D33-Pad1) -> Net-(D53-Pad1)
- SW54 pad 1: Net-(D41-Pad1) -> Net-(D54-Pad1)
- SW55 pad 1: Net-(D60-Pad1) -> Net-(D55-Pad1)
- SW56 pad 1: Net-(D59-Pad1) -> Net-(D56-Pad1)
- SW57 pad 1: Net-(D58-Pad1) -> Net-(D57-Pad1)
- SW58 pad 1: Net-(D48-Pad1) -> Net-(D58-Pad1)
- SW59 pad 1: Net-(D56-Pad1) -> Net-(D59-Pad1)
- SW6 pad 1: Net-(D21-Pad1) -> Net-(D6-Pad1)
- SW60 pad 1: Net-(D49-Pad1) -> Net-(D60-Pad1)
- SW61 pad 1: Net-(D50-Pad1) -> Net-(D61-Pad1)
- SW62 pad 1: Net-(D51-Pad1) -> Net-(D62-Pad1)
- SW63 pad 1: Net-(D52-Pad1) -> Net-(D63-Pad1)
- SW7 pad 1: Net-(D13-Pad1) -> Net-(D7-Pad1)
- SW8 pad 1: Net-(D5-Pad1) -> Net-(D8-Pad1)
- SW9 pad 1: Net-(D4-Pad1) -> Net-(D9-Pad1)
- U1 pad 10: Row3 -> Row2
- U1 pad 11: Row4 -> Row1
- U1 pad 8: Row1 -> Row4
- U1 pad 9: Row2 -> Row3
Routing:
- net Col4: track 0.00 -> 282.4 mm
- net Row4: track 0.00 -> 245.9 mm, vias 0 -> 1
- net Col3: track 0.00 -> 243.5 mm
- net Row3: track 0.00 -> 233.5 mm, vias 0 -> 1
- net Col7: track 0.00 -> 233.3 mm
- net Row2: track 0.00 -> 222.4 mm, vias 0 -> 1
- net Col2: track 0.00 -> 205.0 mm
- net Row5: track 0.00 -> 190.9 mm, vias 0 -> 1
- net Row8: track 0.00 -> 183.0 mm, vias 0 -> 1
- net Row6: track 0.00 -> 174.6 mm, vias 0 -> 1
- net Row7: track 0.00 -> 171.3 mm, vias 0 -> 1
- net Col6: track 0.00 -> 165.2 mm
- net Col1: track 0.00 -> 165.1 mm
- net Col8: track 0.00 -> 159.7 mm
- net Col5: track 0.00 -> 126.1 mm
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- added copper zone on B.Cu, net GND
- added copper zone on F.Cu, net GND
Other:
- outline, holes or cut-outs redrawn
- board text added: "Kibo"
- board text added: "ONE."

Commit message: Work work work
Parts:
- moved C2 18.3 mm to (203.6, 161.2), turned to 180 degrees
- moved Y1 16.6 mm to (205.7, 165.0), turned to 180 degrees
- moved C1 15.3 mm to (208.0, 161.2), turned to 0 degrees
- moved SW_RESET1 8.03 mm to (188.6, 164.5)
- moved R3 6.80 mm to (188.6, 158.8), turned to 180 degrees
Routing:
- net Col7: track 233.3 -> 770.6 mm
- net Col6: track 165.2 -> 542.3 mm
- net Col5: track 126.1 -> 462.5 mm
- net Row1: track 121.1 -> 424.9 mm
- net Row4: track 245.9 -> 510.7 mm
- net Row3: track 233.5 -> 453.6 mm
- net Row2: track 222.4 -> 392.3 mm
- net Col8: track 159.7 -> 312.2 mm
- net Col4: track 282.4 -> 381.4 mm
- net Col3: track 243.5 -> 314.9 mm
- net Col2: track 205.0 -> 268.6 mm
- net Col1: track 165.1 -> 204.3 mm
- net RESET: track 0.00 -> 17.3 mm
- net VBUS: track 73.6 -> 87.6 mm
- net Net-(C1-Pad1): track 8.57 -> 19.5 mm, vias 0 -> 2
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Other:
- board size 304.8 x 100 mm -> 304.8 x 102.4 mm
- net class Cols added: clearance 0.2, trace_width 0.4, via_dia 1, via_drill 0.4
- net class Rows added: clearance 0.2, trace_width 0.4, via_dia 1, via_drill 0.4

Commit message: Various faffing about
Parts:
- moved SW_RESET1 18.7 mm to (207.3, 165.1)
- moved C2 17.9 mm to (186.2, 156.8), turned to 225 degrees
- moved Y1 17.6 mm to (189.0, 159.8), turned to 135 degrees
- moved C1 16.1 mm to (192.0, 162.4), turned to 225 degrees
- moved R3 15.9 mm to (203.2, 165.1)
- moved D49 7.53 mm to (171.4, 162.6), turned to 90 degrees
- moved D10 7.35 mm to (157.2, 104.8), turned to 90 degrees
- moved D17 7.35 mm to (304.8, 123.8), turned to 90 degrees
- moved D18 7.35 mm to (285.8, 123.8), turned to 90 degrees
- moved D19 7.35 mm to (266.7, 123.8), turned to 90 degrees
- moved D2 7.35 mm to (328.6, 104.8), turned to 90 degrees
- moved D21 7.35 mm to (228.6, 123.8), turned to 90 degrees
- moved D23 7.35 mm to (181.0, 123.8), turned to 90 degrees
- moved D25 7.35 mm to (142.9, 123.8), turned to 90 degrees
- moved D29 7.35 mm to (338.1, 142.9), turned to 90 degrees
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Connections:
- D1 pad 1: Net-(D1-Pad1) -> Col8
- D1 pad 2: Row5 -> Net-(D1-Pad2)
- D10 pad 1: Net-(D10-Pad1) -> Col2
- D10 pad 2: Row4 -> Net-(D10-Pad2)
- D11 pad 1: Net-(D11-Pad1) -> Col3
- D11 pad 2: Row4 -> Net-(D11-Pad2)
- D12 pad 1: Net-(D12-Pad1) -> Col4
- D12 pad 2: Row4 -> Net-(D12-Pad2)
- D13 pad 1: Net-(D13-Pad1) -> Col5
- D13 pad 2: Row4 -> Net-(D13-Pad2)
- D14 pad 1: Net-(D14-Pad1) -> Col6
- D14 pad 2: Row4 -> Net-(D14-Pad2)
- D15 pad 1: Net-(D15-Pad1) -> Col8
- D15 pad 2: Row6 -> Net-(D15-Pad2)
- D16 pad 1: Net-(D16-Pad1) -> Col7
- D16 pad 2: Row6 -> Net-(D16-Pad2)
- D17 pad 1: Net-(D17-Pad1) -> Col6
- D17 pad 2: Row6 -> Net-(D17-Pad2)
- D18 pad 1: Net-(D18-Pad1) -> Col5
- D18 pad 2: Row6 -> Net-(D18-Pad2)
- D19 pad 1: Net-(D19-Pad1) -> Col4
- D19 pad 2: Row6 -> Net-(D19-Pad2)
- D2 pad 1: Net-(D2-Pad1) -> Col7
- D2 pad 2: Row5 -> Net-(D2-Pad2)
- D20 pad 1: Net-(D20-Pad1) -> Col3
- D20 pad 2: Row6 -> Net-(D20-Pad2)
- D21 pad 1: Net-(D21-Pad1) -> Col2
- D21 pad 2: Row6 -> Net-(D21-Pad2)
- D22 pad 1: Net-(D22-Pad1) -> Col1
- D22 pad 2: Row6 -> Net-(D22-Pad2)
- D23 pad 1: Net-(D23-Pad1) -> Col1
- D23 pad 2: Row3 -> Net-(D23-Pad2)
- D24 pad 1: Net-(D24-Pad1) -> Col2
- D24 pad 2: Row3 -> Net-(D24-Pad2)
- D25 pad 1: Net-(D25-Pad1) -> Col3
- D25 pad 2: Row3 -> Net-(D25-Pad2)
- D26 pad 1: Net-(D26-Pad1) -> Col4
- D26 pad 2: Row3 -> Net-(D26-Pad2)
- D27 pad 1: Net-(D27-Pad1) -> Col5
- D27 pad 2: Row3 -> Net-(D27-Pad2)
- D28 pad 1: Net-(D28-Pad1) -> Col6
- D28 pad 2: Row3 -> Net-(D28-Pad2)
- D29 pad 1: Net-(D29-Pad1) -> Col7
- D29 pad 2: Row7 -> Net-(D29-Pad2)
- D3 pad 1: Net-(D3-Pad1) -> Col6
- D3 pad 2: Row5 -> Net-(D3-Pad2)
- D30 pad 1: Net-(D30-Pad1) -> Col6
- D30 pad 2: Row7 -> Net-(D30-Pad2)
- D31 pad 1: Net-(D31-Pad1) -> Col5
- D31 pad 2: Row7 -> Net-(D31-Pad2)
- D32 pad 1: Net-(D32-Pad1) -> Col4
- D32 pad 2: Row7 -> Net-(D32-Pad2)
- D33 pad 1: Net-(D33-Pad1) -> Col3
- D33 pad 2: Row7 -> Net-(D33-Pad2)
- D34 pad 1: Net-(D34-Pad1) -> Col2
- D34 pad 2: Row7 -> Net-(D34-Pad2)
- D35 pad 1: Net-(D35-Pad1) -> Col1
- D35 pad 2: Row7 -> Net-(D35-Pad2)
- D36 pad 1: Net-(D36-Pad1) -> Col1
- D36 pad 2: Row2 -> Net-(D36-Pad2)
- D37 pad 1: Net-(D37-Pad1) -> Col2
- D37 pad 2: Row2 -> Net-(D37-Pad2)
- D38 pad 1: Net-(D38-Pad1) -> Col3
- D38 pad 2: Row2 -> Net-(D38-Pad2)
- D39 pad 1: Net-(D39-Pad1) -> Col4
- D39 pad 2: Row2 -> Net-(D39-Pad2)
- D4 pad 1: Net-(D4-Pad1) -> Col5
- D4 pad 2: Row5 -> Net-(D4-Pad2)
- D40 pad 1: Net-(D40-Pad1) -> Col5
- D40 pad 2: Row2 -> Net-(D40-Pad2)
- D41 pad 1: Net-(D41-Pad1) -> Col6
- D41 pad 2: Row2 -> Net-(D41-Pad2)
- D42 pad 1: Net-(D42-Pad1) -> Col8
- D42 pad 2: Row7 -> Net-(D42-Pad2)
- D43 pad 1: Net-(D43-Pad1) -> Col8
- D43 pad 2: Row1 -> Net-(D43-Pad2)
- D44 pad 1: Net-(D44-Pad1) -> Col5
- D44 pad 2: Row8 -> Net-(D44-Pad2)
- D45 pad 1: Net-(D45-Pad1) -> Col4
- D45 pad 2: Row8 -> Net-(D45-Pad2)
- D46 pad 1: Net-(D46-Pad1) -> Col3
- D46 pad 2: Row8 -> Net-(D46-Pad2)
- D47 pad 1: Net-(D47-Pad1) -> Col2
- D47 pad 2: Row8 -> Net-(D47-Pad2)
- D48 pad 1: Net-(D48-Pad1) -> Col1
- D48 pad 2: Row8 -> Net-(D48-Pad2)
- D49 pad 1: Net-(D49-Pad1) -> Col1
- D49 pad 2: Row1 -> Net-(D49-Pad2)
- D5 pad 1: Net-(D5-Pad1) -> Col4
- D5 pad 2: Row5 -> Net-(D5-Pad2)
- D50 pad 1: Net-(D50-Pad1) -> Col2
- D50 pad 2: Row1 -> Net-(D50-Pad2)
- D51 pad 1: Net-(D51-Pad1) -> Col3
- D51 pad 2: Row1 -> Net-(D51-Pad2)
- D52 pad 1: Net-(D52-Pad1) -> Col4
- D52 pad 2: Row1 -> Net-(D52-Pad2)
- D53 pad 1: Net-(D53-Pad1) -> Col5
- D53 pad 2: Row1 -> Net-(D53-Pad2)
- D54 pad 1: Net-(D54-Pad1) -> Col6
- D54 pad 2: Row1 -> Net-(D54-Pad2)
- D55 pad 1: Net-(D55-Pad1) -> Col8
- D55 pad 2: Row4 -> Net-(D55-Pad2)
- D56 pad 1: Net-(D56-Pad1) -> Col8
- D56 pad 2: Row3 -> Net-(D56-Pad2)
- D57 pad 1: Net-(D57-Pad1) -> Col8
- D57 pad 2: Row2 -> Net-(D57-Pad2)
- D58 pad 1: Net-(D58-Pad1) -> Col6
- D58 pad 2: Row8 -> Net-(D58-Pad2)
- D59 pad 1: Net-(D59-Pad1) -> Col7
- D59 pad 2: Row8 -> Net-(D59-Pad2)
- D6 pad 1: Net-(D6-Pad1) -> Col3
- D6 pad 2: Row5 -> Net-(D6-Pad2)
- D60 pad 1: Net-(D60-Pad1) -> Col7
- D60 pad 2: Row1 -> Net-(D60-Pad2)
- D61 pad 1: Net-(D61-Pad1) -> Col7
- D61 pad 2: Row2 -> Net-(D61-Pad2)
- D62 pad 1: Net-(D62-Pad1) -> Col7
- D62 pad 2: Row3 -> Net-(D62-Pad2)
- D63 pad 1: Net-(D63-Pad1) -> Col7
- D63 pad 2: Row4 -> Net-(D63-Pad2)
- D7 pad 1: Net-(D7-Pad1) -> Col2
- D7 pad 2: Row5 -> Net-(D7-Pad2)
- D8 pad 1: Net-(D8-Pad1) -> Col1
- D8 pad 2: Row5 -> Net-(D8-Pad2)
- D9 pad 1: Net-(D9-Pad1) -> Col1
- D9 pad 2: Row4 -> Net-(D9-Pad2)
- SW1 pad 1: Net-(D1-Pad1) -> Row5
- SW1 pad 2: Col8 -> Net-(D1-Pad2)
- SW10 pad 1: Net-(D10-Pad1) -> Row4
- SW10 pad 2: Col2 -> Net-(D10-Pad2)
- SW11 pad 1: Net-(D11-Pad1) -> Row4
- SW11 pad 2: Col3 -> Net-(D11-Pad2)
- SW12 pad 1: Net-(D12-Pad1) -> Row4
- SW12 pad 2: Col4 -> Net-(D12-Pad2)
- SW13 pad 1: Net-(D13-Pad1) -> Row4
- SW13 pad 2: Col5 -> Net-(D13-Pad2)
- SW14 pad 1: Net-(D14-Pad1) -> Row4
- SW14 pad 2: Col6 -> Net-(D14-Pad2)
- SW15 pad 1: Net-(D15-Pad1) -> Row6
- SW15 pad 2: Col8 -> Net-(D15-Pad2)
- SW16 pad 1: Net-(D16-Pad1) -> Row6
- SW16 pad 2: Col7 -> Net-(D16-Pad2)
- SW17 pad 1: Net-(D17-Pad1) -> Row6
- SW17 pad 2: Col6 -> Net-(D17-Pad2)
- SW18 pad 1: Net-(D18-Pad1) -> Row6
- SW18 pad 2: Col5 -> Net-(D18-Pad2)
- SW19 pad 1: Net-(D19-Pad1) -> Row6
- SW19 pad 2: Col4 -> Net-(D19-Pad2)
- SW2 pad 1: Net-(D2-Pad1) -> Row5
- SW2 pad 2: Col7 -> Net-(D2-Pad2)
- SW20 pad 1: Net-(D20-Pad1) -> Row6
- SW20 pad 2: Col3 -> Net-(D20-Pad2)
- SW21 pad 1: Net-(D21-Pad1) -> Row6
- SW21 pad 2: Col2 -> Net-(D21-Pad2)
- SW22 pad 1: Net-(D22-Pad1) -> Row6
- SW22 pad 2: Col1 -> Net-(D22-Pad2)
- SW23 pad 1: Net-(D23-Pad1) -> Row3
- SW23 pad 2: Col1 -> Net-(D23-Pad2)
- SW24 pad 1: Net-(D24-Pad1) -> Row3
- SW24 pad 2: Col2 -> Net-(D24-Pad2)
- SW25 pad 1: Net-(D25-Pad1) -> Row3
- SW25 pad 2: Col3 -> Net-(D25-Pad2)
- SW26 pad 1: Net-(D26-Pad1) -> Row3
- SW26 pad 2: Col4 -> Net-(D26-Pad2)
- SW27 pad 1: Net-(D27-Pad1) -> Row3
- SW27 pad 2: Col5 -> Net-(D27-Pad2)
- SW28 pad 1: Net-(D28-Pad1) -> Row3
- SW28 pad 2: Col6 -> Net-(D28-Pad2)
- SW29 pad 1: Net-(D29-Pad1) -> Row7
- SW29 pad 2: Col7 -> Net-(D29-Pad2)
- SW3 pad 1: Net-(D3-Pad1) -> Row5
- SW3 pad 2: Col6 -> Net-(D3-Pad2)
- SW30 pad 1: Net-(D30-Pad1) -> Row7
- SW30 pad 2: Col6 -> Net-(D30-Pad2)
- SW31 pad 1: Net-(D31-Pad1) -> Row7
- SW31 pad 2: Col5 -> Net-(D31-Pad2)
- SW32 pad 1: Net-(D32-Pad1) -> Row7
- SW32 pad 2: Col4 -> Net-(D32-Pad2)
- SW33 pad 1: Net-(D33-Pad1) -> Row7
- SW33 pad 2: Col3 -> Net-(D33-Pad2)
- SW34 pad 1: Net-(D34-Pad1) -> Row7
- SW34 pad 2: Col2 -> Net-(D34-Pad2)
- SW35 pad 1: Net-(D35-Pad1) -> Row7
- SW35 pad 2: Col1 -> Net-(D35-Pad2)
- SW36 pad 1: Net-(D36-Pad1) -> Row2
- SW36 pad 2: Col1 -> Net-(D36-Pad2)
- SW37 pad 1: Net-(D37-Pad1) -> Row2
- SW37 pad 2: Col2 -> Net-(D37-Pad2)
- SW38 pad 1: Net-(D38-Pad1) -> Row2
- SW38 pad 2: Col3 -> Net-(D38-Pad2)
- SW39 pad 1: Net-(D39-Pad1) -> Row2
- SW39 pad 2: Col4 -> Net-(D39-Pad2)
- SW4 pad 1: Net-(D4-Pad1) -> Row5
- SW4 pad 2: Col5 -> Net-(D4-Pad2)
- SW40 pad 1: Net-(D40-Pad1) -> Row2
- SW40 pad 2: Col5 -> Net-(D40-Pad2)
- SW41 pad 1: Net-(D41-Pad1) -> Row2
- SW41 pad 2: Col6 -> Net-(D41-Pad2)
- SW42 pad 1: Net-(D42-Pad1) -> Row7
- SW42 pad 2: Col8 -> Net-(D42-Pad2)
- SW43 pad 1: Net-(D43-Pad1) -> Row1
- SW43 pad 2: Col8 -> Net-(D43-Pad2)
- SW44 pad 1: Net-(D44-Pad1) -> Row8
- SW44 pad 2: Col5 -> Net-(D44-Pad2)
- SW45 pad 1: Net-(D45-Pad1) -> Row8
- SW45 pad 2: Col4 -> Net-(D45-Pad2)
- SW46 pad 1: Net-(D46-Pad1) -> Row8
- SW46 pad 2: Col3 -> Net-(D46-Pad2)
- SW47 pad 1: Net-(D47-Pad1) -> Row8
- SW47 pad 2: Col2 -> Net-(D47-Pad2)
- SW48 pad 1: Net-(D48-Pad1) -> Row8
- SW48 pad 2: Col1 -> Net-(D48-Pad2)
- SW49 pad 1: Net-(D49-Pad1) -> Row1
- SW49 pad 2: Col1 -> Net-(D49-Pad2)
- SW5 pad 1: Net-(D5-Pad1) -> Row5
- SW5 pad 2: Col4 -> Net-(D5-Pad2)
- SW50 pad 1: Net-(D50-Pad1) -> Row1
- SW50 pad 2: Col2 -> Net-(D50-Pad2)
- SW51 pad 1: Net-(D51-Pad1) -> Row1
- SW51 pad 2: Col3 -> Net-(D51-Pad2)
- SW52 pad 1: Net-(D52-Pad1) -> Row1
- SW52 pad 2: Col4 -> Net-(D52-Pad2)
- SW53 pad 1: Net-(D53-Pad1) -> Row1
- SW53 pad 2: Col5 -> Net-(D53-Pad2)
- SW54 pad 1: Net-(D54-Pad1) -> Row1
- SW54 pad 2: Col6 -> Net-(D54-Pad2)
- SW55 pad 1: Net-(D55-Pad1) -> Row4
- SW55 pad 2: Col8 -> Net-(D55-Pad2)
- SW56 pad 1: Net-(D56-Pad1) -> Row3
- SW56 pad 2: Col8 -> Net-(D56-Pad2)
- SW57 pad 1: Net-(D57-Pad1) -> Row2
- SW57 pad 2: Col8 -> Net-(D57-Pad2)
- SW58 pad 1: Net-(D58-Pad1) -> Row8
- SW58 pad 2: Col6 -> Net-(D58-Pad2)
- SW59 pad 1: Net-(D59-Pad1) -> Row8
- SW59 pad 2: Col7 -> Net-(D59-Pad2)
- SW6 pad 1: Net-(D6-Pad1) -> Row5
- SW6 pad 2: Col3 -> Net-(D6-Pad2)
- SW60 pad 1: Net-(D60-Pad1) -> Row1
- SW60 pad 2: Col7 -> Net-(D60-Pad2)
- SW61 pad 1: Net-(D61-Pad1) -> Row2
- SW61 pad 2: Col7 -> Net-(D61-Pad2)
- SW62 pad 1: Net-(D62-Pad1) -> Row3
- SW62 pad 2: Col7 -> Net-(D62-Pad2)
- SW63 pad 1: Net-(D63-Pad1) -> Row4
- SW63 pad 2: Col7 -> Net-(D63-Pad2)
- SW7 pad 1: Net-(D7-Pad1) -> Row5
- SW7 pad 2: Col2 -> Net-(D7-Pad2)
- SW8 pad 1: Net-(D8-Pad1) -> Row5
- SW8 pad 2: Col1 -> Net-(D8-Pad2)
- SW9 pad 1: Net-(D9-Pad1) -> Row4
- SW9 pad 2: Col1 -> Net-(D9-Pad2)
Routing:
- net Col6: track 542.3 -> 110.8 mm
- net Col7: track 770.6 -> 371.3 mm, vias 0 -> 3
- net Col5: track 462.5 -> 131.9 mm
- net Col3: track 314.9 -> 131.4 mm
- net Col4: track 381.4 -> 213.5 mm, vias 0 -> 1
- net Col8: track 312.2 -> 152.4 mm
- net Row1: track 424.9 -> 293.6 mm
- net Row5: track 190.9 -> 270.5 mm, vias 1 -> 0
- net Row6: track 174.6 -> 249.1 mm, vias 1 -> 0
- net Col2: track 268.6 -> 195.8 mm, vias 0 -> 3
- net Col1: track 204.3 -> 158.2 mm, vias 0 -> 1
- net Row4: track 510.7 -> 553.9 mm, vias 1 -> 0
- net Row7: track 171.3 -> 212.6 mm, vias 1 -> 0
- net Row8: track 173.8 -> 146.9 mm, vias 1 -> 0
- net RESET: track 17.3 -> 0.00 mm
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Other:
- board size 304.8 x 102.4 mm -> 304.8 x 100 mm
- net class Cols: clearance 0.2 -> 0.3
- net class Rows: clearance 0.2 -> 0.3

Commit message: Prep for dual-board design
Parts:
- moved SW_RESET1 4.81 mm to (206.1, 160.4), turned to 45 degrees
- moved R3 2.28 mm to (201.2, 164.1), turned to 315 degrees
Routing:
- net Col2: track 195.8 -> 179.2 mm
- net Col1: track 158.2 -> 143.9 mm
- net Col4: track 213.5 -> 200.5 mm, vias 1 -> 2
- net Row4: track 553.9 -> 541.6 mm, vias 0 -> 1
- net Row3: track 466.4 -> 455.2 mm, vias 0 -> 1
- net Row8: track 146.9 -> 138.7 mm, vias 0 -> 1
- net Row7: track 212.6 -> 204.8 mm, vias 0 -> 1
- net GND: track 23.9 -> 18.8 mm
- net Row2: track 381.2 -> 377.8 mm, vias 0 -> 1
- net D+: track 14.7 -> 17.6 mm
- net D-: track 12.6 -> 14.8 mm, vias 0 -> 2
- net Row6: vias 0 -> 1
- net Row5: vias 0 -> 1
Other:
- board text added: "Kullen"
- board text added: "Robotics"
